Commit message: fix the hips of the dog

File: uniteedog_description/urdf/unitreeDog.urdf (robot description, URDF)
Before this commit: robot UnitreeDog, 12 links, 11 joints
Links:
- removed link hip
- added link back_hip_left; visual mesh filename=package://uniteedog_description/meshes/hip.dae scale=1.0 1.0 1.0
- added link back_hip_right; visual mesh filename=package://uniteedog_description/meshes/hip.dae scale=1.0 1.0 1.0
- added link front_hip_left; visual mesh filename=package://uniteedog_description/meshes/hip.dae scale=1.0 1.0 1.0
- added link front_hip_right; visual mesh filename=package://uniteedog_description/meshes/hip.dae scale=1.0 1.0 1.0
Joints:
- removed joint base_to_hip
- added joint base_to_back_hip_left: type revolute, parent base_link, child back_hip_left, origin xyz=-0.19 0.05 0 rpy=0 0 0, axis 1 0 0, limit lower=-0.6 upper=0.6 effort=10 velocity=0.5
- added joint base_to_back_hip_right: type revolute, parent base_link, child back_hip_right, origin xyz=-0.19 -0.05 0 rpy=0 0 0, axis 1 0 0, limit lower=-0.6 upper=0.6 effort=10 velocity=0.5
- added joint base_to_front_hip_left: type revolute, parent base_link, child front_hip_left, origin xyz=0.19 0.05 0 rpy=0 0 0, axis 1 0 0, limit lower=-0.6 upper=0.6 effort=10 velocity=0.5
- added joint base_to_front_hip_right: type revolute, parent base_link, child front_hip_right, origin xyz=0.19 -0.05 0 rpy=0 0 0, axis 1 0 0, limit lower=-0.6 upper=0.6 effort=10 velocity=0.5
- joint base_to_left_front_leg: axis (none) -> 0 1 0; limit (none) -> lower=-0.52 upper=1.57 effort=10 velocity=0.5; origin xyz=0.18 0.1 0  rpy=0 0 0 -> xyz=0 0.08 0  rpy=0 0 0; parent base_link -> front_hip_left; type fixed -> revolute
- joint base_to_right_front_leg: axis (none) -> 0 1 0; limit (none) -> lower=-0.52 upper=1.57 effort=10 velocity=0.5; origin xyz=0.18 -0.1 0  rpy=0 0 0 -> xyz=0 -0.08 0  rpy=0 0 0; parent base_link -> front_hip_right; type fixed -> revolute
- joint hip_to_left_back_leg: axis (none) -> 0 1 0; limit (none) -> lower=-0.52 upper=1.57 effort=10 velocity=0.5; parent hip -> back_hip_left; type fixed -> revolute
- joint hip_to_right_back_leg: axis (none) -> 0 1 0; limit (none) -> lower=-0.52 upper=1.57 effort=10 velocity=0.5; parent hip -> back_hip_right; type fixed -> revolute
- joint left_back_leg_to_calf: axis (none) -> 0 1 0; limit (none) -> lower=-1.2 upper=0 effort=10 velocity=0.5; type fixed -> revolute
- joint left_front_leg_to_calf: axis (none) -> 0 1 0; limit (none) -> lower=-1.2 upper=0 effort=10 velocity=0.5; type fixed -> revolute
- joint right_back_leg_to_calf: axis (none) -> 0 1 0; limit (none) -> lower=-1.2 upper=0 effort=10 velocity=0.5; type fixed -> revolute
- joint right_front_leg_to_calf: axis (none) -> 0 1 0; limit (none) -> lower=-1.2 upper=0 effort=10 velocity=0.5; type fixed -> revolute
