Commit message: Edited the launch file to bringup gazebo

File: uniteedog_description/urdf/unitreeDog.urdf.xacro (robot description, xacro)
@@ -1,3 +1,3 @@
-<robot name="UnitreeDog">
+<robot name="UnitreeDog" xmlns:xacro="http://www.ros.org/wiki/xacro">
   <!-- ===========================
        BASE / TRUNK (box approx)
@@ -21,5 +21,5 @@
     </collision>
     <!-- Inertial: computed for the box geometry -->
-    <inertial>
+    <!-- <inertial>
       <origin xyz="0 0 0" rpy="0 0 0"/>
       <mass value="5.5"/>
@@ -28,5 +28,5 @@
         iyy="0.16506600" iyz="0.0"
         izz="0.18064933"/>
-    </inertial>
+    </inertial> -->
   </link>
   <!-- ===========================
@@ -198,4 +198,26 @@
         izz="0.000054"/>
     </inertial>
+    <sensor name="unitree_camera" type="camera">
+    <pose>0 0 0 0 0 0</pose>
+    <visualize>true</visualize>
+    <update_rate>30</update_rate>
+    <camera>
+      <horizontal_fov>1.089</horizontal_fov>
+      <image>
+        <width>640</width>
+        <height>480</height>
+        <format>R8G8B8</format>
+      </image>
+      <clip>
+        <near>0.05</near>
+        <far>8.0</far>
+      </clip>
+    </camera>
+    <topic>camera/image_raw</topic>
+    <plugin
+      filename="ignition-gazebo-camera-plugin"
+      name="ignition::gazebo::systems::Camera">
+    </plugin>
+  </sensor>
   </link>
   <joint name="base_to_camera" type="fixed">
@@ -511,5 +533,5 @@
     <origin xyz="-0.14 0 -0.15" rpy="0 -0.7854 0"/>
   </joint>
-  <gazebo>
+  <!-- <gazebo>
   <plugin name="ros2_control" filename="libignition_ros2_control.so">
     <ros2_control>
@@ -526,4 +548,18 @@
     <updateRate>30</updateRate>
   </plugin>
+</gazebo> -->
+<gazebo>
+  <plugin
+    filename="ign_ros2_control-system"
+    name="ign_ros2_control::IgnitionRos2ControlSystem">
+    <ros>
+      <namespace>/</namespace>
+    </ros>
+    </plugin>
+  <plugin
+    filename="ignition-gazebo-sensors-system"
+    name="ignition::gazebo::systems::Sensors">
+    <render_engine>ogre2</render_engine>
+  </plugin>
 </gazebo>
 </robot>
