Commit message: Fix bug caused by incorrect renaming

File: unitreedog_description/urdf/unitreeDog.urdf.xacro (robot description, xacro)
@@ -7,5 +7,5 @@
       <origin xyz="0 0 0" rpy="0 0 0"/>
       <geometry>
-        <mesh filename="package://uniteedog_description/meshes/trunk.dae" scale="1.0 1.0 1.0"/>
+        <mesh filename="package://unitreedog_description/meshes/trunk.dae" scale="1.0 1.0 1.0"/>
       </geometry>
       <material name="base_color">
@@ -37,5 +37,5 @@
       <origin xyz="0 0 0" rpy="0 3.1416 0"/>
       <geometry>
-        <mesh filename="package://uniteedog_description/meshes/hip.dae" scale="1.0 1.0 1.0"/>
+        <mesh filename="package://unitreedog_description/meshes/hip.dae" scale="1.0 1.0 1.0"/>
       </geometry>
       <material name="base_color">
@@ -72,5 +72,5 @@
       <origin xyz="0 0 0" rpy="0 3.1416 0"/>
       <geometry>
-        <mesh filename="package://uniteedog_description/meshes/hip.dae" scale="1.0 1.0 1.0"/>
+        <mesh filename="package://unitreedog_description/meshes/hip.dae" scale="1.0 1.0 1.0"/>
       </geometry>
       <material name="base_color">
@@ -107,5 +107,5 @@
       <origin xyz="0 0 0" rpy="0 0 0"/>
       <geometry>
-        <mesh filename="package://uniteedog_description/meshes/hip.dae" scale="1.0 1.0 1.0"/>
+        <mesh filename="package://unitreedog_description/meshes/hip.dae" scale="1.0 1.0 1.0"/>
       </geometry>
       <material name="base_color">
@@ -142,5 +142,5 @@
       <origin xyz="0 0 0" rpy="0 0 0"/>
       <geometry>
-        <mesh filename="package://uniteedog_description/meshes/hip.dae" scale="1.0 1.0 1.0"/>
+        <mesh filename="package://unitreedog_description/meshes/hip.dae" scale="1.0 1.0 1.0"/>
       </geometry>
       <material name="base_color">
@@ -177,5 +177,5 @@
       <origin xyz="0 -0.01 0.01" rpy="0.7854 0 0"/>
       <geometry>
-        <mesh filename="package://uniteedog_description/meshes/depthCamera.dae" scale="1.0 1.0 1.0"/>
+        <mesh filename="package://unitreedog_description/meshes/depthCamera.dae" scale="1.0 1.0 1.0"/>
       </geometry>
       <material name="base_color">
@@ -233,5 +233,5 @@
       <origin xyz="0 0 0.02" rpy="-0.7854 0 0"/>
       <geometry>
-        <mesh filename="package://uniteedog_description/meshes/ultraSound.dae" scale="1.0 1.0 1.0"/>
+        <mesh filename="package://unitreedog_description/meshes/ultraSound.dae" scale="1.0 1.0 1.0"/>
       </geometry>
       <material name="base_color">
@@ -266,5 +266,5 @@
       <origin xyz="0 0 0" rpy="0 0.7854 0"/>
       <geometry>
-        <mesh filename="package://uniteedog_description/meshes/thigh_mirror.dae" scale="1.0 1.0 1.0"/>
+        <mesh filename="package://unitreedog_description/meshes/thigh_mirror.dae" scale="1.0 1.0 1.0"/>
       </geometry>
       <material name="base_color">
@@ -301,5 +301,5 @@
       <origin xyz="0 0 0" rpy="0 0 0"/>
       <geometry>
-        <mesh filename="package://uniteedog_description/meshes/calf.dae" scale="1.0 1.0 1.0"/>
+        <mesh filename="package://unitreedog_description/meshes/calf.dae" scale="1.0 1.0 1.0"/>
       </geometry>
       <material name="base_color">
@@ -339,5 +339,5 @@
       <origin xyz="0 0 0" rpy="0 0.7854 0"/>
       <geometry>
-        <mesh filename="package://uniteedog_description/meshes/thigh.dae" scale="1.0 1.0 1.0"/>
+        <mesh filename="package://unitreedog_description/meshes/thigh.dae" scale="1.0 1.0 1.0"/>
       </geometry>
       <material name="base_color">
@@ -371,5 +371,5 @@
       <origin xyz="0 0 0" rpy="0 0 0"/>
       <geometry>
-        <mesh filename="package://uniteedog_description/meshes/calf.dae" scale="1.0 1.0 1.0"/>
+        <mesh filename="package://unitreedog_description/meshes/calf.dae" scale="1.0 1.0 1.0"/>
       </geometry>
       <material name="base_color">
@@ -406,5 +406,5 @@
       <origin xyz="0 0 0" rpy="0 0.7854 0"/>
       <geometry>
-        <mesh filename="package://uniteedog_description/meshes/thigh_mirror.dae" scale="1.0 1.0 1.0"/>
+        <mesh filename="package://unitreedog_description/meshes/thigh_mirror.dae" scale="1.0 1.0 1.0"/>
       </geometry>
       <material name="base_color">
@@ -438,5 +438,5 @@
       <origin xyz="0 0 0" rpy="0 0 0"/>
       <geometry>
-        <mesh filename="package://uniteedog_description/meshes/calf.dae" scale="1.0 1.0 1.0"/>
+        <mesh filename="package://unitreedog_description/meshes/calf.dae" scale="1.0 1.0 1.0"/>
       </geometry>
       <material name="base_color">
@@ -473,5 +473,5 @@
       <origin xyz="0 0 0" rpy="0 0.7854 0"/>
       <geometry>
-        <mesh filename="package://uniteedog_description/meshes/thigh.dae" scale="1.0 1.0 1.0"/>
+        <mesh filename="package://unitreedog_description/meshes/thigh.dae" scale="1.0 1.0 1.0"/>
       </geometry>
       <material name="base_color">
@@ -505,5 +505,5 @@
       <origin xyz="0 0 0" rpy="0 0 0"/>
       <geometry>
-        <mesh filename="package://uniteedog_description/meshes/calf.dae" scale="1.0 1.0 1.0"/>
+        <mesh filename="package://unitreedog_description/meshes/calf.dae" scale="1.0 1.0 1.0"/>
       </geometry>
       <material name="base_color">
